Commit message: (feat): home position and basic code configuration

File: agrirover_description/urdf/mech/arm_combined.urdf (robot description, URDF)
Before this commit: robot arm, 9 links, 8 joints
Links:
- added link camera_head_color_frame
- added link camera_head_color_optical_frame
- added link camera_head_depth_frame
- added link camera_head_depth_optical_frame
- added link camera_head_infra1_frame
- added link camera_head_infra1_optical_frame
- added link camera_head_infra2_frame
- added link camera_head_infra2_optical_frame
- added link camera_head_link, mass 0.072; collision box size=0.02505 0.090 0.025; visual mesh filename=package://agrirover_description/meshes/d435/visual/d435.stl
Joints:
- added joint camera_head_color_joint: type fixed, parent camera_head_link, child camera_head_color_frame, origin xyz=0 0.015 0 rpy=0 0 0
- added joint camera_head_color_optical_joint: type fixed, parent camera_head_color_frame, child camera_head_color_optical_frame, origin xyz=0 0 0 rpy=-1.5707963267948966 0 -1.5707963267948966
- added joint camera_head_depth_joint: type fixed, parent camera_head_link, child camera_head_depth_frame, origin xyz=0 0 0 rpy=0 0 0
- added joint camera_head_depth_optical_joint: type fixed, parent camera_head_depth_frame, child camera_head_depth_optical_frame, origin xyz=0 0 0 rpy=-1.5707963267948966 0 -1.5707963267948966
- added joint camera_head_infra1_joint: type fixed, parent camera_head_link, child camera_head_infra1_frame, origin xyz=0 0.0 0 rpy=0 0 0
- added joint camera_head_infra1_optical_joint: type fixed, parent camera_head_infra1_frame, child camera_head_infra1_optical_frame, origin xyz=0 0 0 rpy=-1.5707963267948966 0 -1.5707963267948966
- added joint camera_head_infra2_joint: type fixed, parent camera_head_link, child camera_head_infra2_frame, origin xyz=0 -0.050 0 rpy=0 0 0
- added joint camera_head_infra2_optical_joint: type fixed, parent camera_head_infra2_frame, child camera_head_infra2_optical_frame, origin xyz=0 0 0 rpy=-1.5707963267948966 0 -1.5707963267948966
- added joint gripper_to_camera: type fixed, parent gripper, child camera_head_link, origin xyz=-0.025 0.02 0 rpy=-1.57 0 1.57

File: agrirover_description/urdf/robots/arm.urdf.xacro (robot description, xacro)
@@ -2,4 +2,9 @@
 <robot name="agrirover" xmlns:xacro="http://www.ros.org/wiki/xacro">
   <xacro:include filename="$(find agrirover_description)/urdf/mech/arm_mech.urdf"/>
-  <xacro:include filename="$(find agrirover_description)/urdf/control/agrirover_ros2_control.urdf.xacro"/>
+  <xacro:include filename="$(find agrirover_description)/urdf/sensors/intel_rgbd_cam_d435.urdf.xacro"/>
+  <joint name="gripper_to_camera" type="fixed">
+  <parent link="gripper"/>
+  <child link="camera_head_link"/>
+  <origin xyz="-0.025 0.02 0" rpy="1.57 0 -1.57"/>
+  </joint>
 </robot>

File: agrirover_description/urdf/sensors/intel_rgbd_cam_d435.urdf.xacro (robot description, xacro)
@@ -13,51 +13,4 @@
     <xacro:property name="d435_cam_depth_to_color_offset" value="0.015"/>
     <xacro:property name="camera_tilt_angle_deg" value="25"/>
-    <link name="torso_link">
-      <inertial>
-        <origin xyz="0 0 0.50" />
-        <mass value="2.5" />
-        <inertia ixx="0.8" ixy="0.0" ixz="0.0" iyy="0.8" iyz="0.0" izz="0.8" />
-      </inertial>
-      <visual name="holder">
-        <origin xyz="0 0 0.25" rpy="0 0 0" />
-        <material name="LightGrey">
-          <color rgba="0.7 0.7 0.7 1.0"/>
-        </material>
-        <geometry>
-          <cylinder radius="0.005" length="0.5"/>
-        </geometry>
-      </visual>
-      <visual name="base">
-        <origin xyz="0 0 0" rpy="0 0 0" />
-        <material name="LightGrey">
-          <color rgba="0.7 0.7 0.7 1.0"/>
-        </material>
-        <geometry>
-          <box size="0.15 0.10 0.06" />
-        </geometry>
-      </visual>
-      <collision name="holder">
-        <origin xyz="0 0 0.25" rpy="0 0 0" />
-        <geometry>
-          <cylinder radius="0.005" length="0.6"/>
-        </geometry>
-      </collision>
-      <collision name="base">
-        <origin xyz="0 0 0.0" rpy="0 0 0" />
-        <geometry>
-          <box size="0.15 0.10 0.06" />
-        </geometry>
-      </collision>
-    </link>
-    <joint name="$(arg prefix)base_link_to_torso_link" type="fixed">
-      <parent link="$(arg prefix)base_link"/>
-      <child link="torso_link"/>
-      <origin xyz="0.22 -0.30 0" rpy="0 0 0"/>
-    </joint>
-    <joint name="camera_head_joint" type="fixed">
-      <parent link="torso_link"/>
-      <child link="camera_head_link" />
-      <origin xyz="0 0.01 0.50" rpy="0.0 ${camera_tilt_angle_deg * M_PI / 180} ${M_PI/2}"/>
-    </joint>
     <link name="camera_head_link">
       <visual>

Commit message: (feat): URDF Corrected

File: agrirover_description/urdf/mech/arm_combined.urdf (robot description, URDF)
Before this commit: robot agrirover, 18 links, 17 joints
Joints:
- joint link_0_to_link_1: axis 0 0 1 -> 0 0 -1; origin xyz=0 0 0.05 rpy=1.57 1.57 0 -> xyz=0 0 0.05 rpy=1.57 -1.57 0
- joint link_1_to_link_2: axis 0 0 1 -> 0 0 -1; origin xyz=0 0.176 0 rpy=0 0 -1.57 -> xyz=0 0.176 0 rpy=0 0 1.57

Commit message: (feat): URDF re-corected

File: agrirover_description/urdf/mech/arm_combined.urdf (robot description, URDF)
Before this commit: robot agrirover, 18 links, 17 joints
Joints:
- joint base_to_link_0: origin xyz=0 0 0.03 rpy=0 0 3.14 -> xyz=0 0 0.03 rpy=0 0 0
- joint link_0_to_link_1: axis 0 0 -1 -> 0 0 1; origin xyz=0 0 0.05 rpy=1.57 -1.57 0 -> xyz=0 0 0.05 rpy=1.57 1.57 0
- joint link_1_to_link_2: axis 0 0 -1 -> 0 0 1; origin xyz=0 0.176 0 rpy=0 0 1.57 -> xyz=0 0.176 0 rpy=0 0 -1.57
